File: test/test_project_bad_table/test_project_bad_table.kicad_sch (KiCad schematic)
At the start: 5 parts

Commit message: Github Actions testing
Parts:
- removed C1: C, Capacitor_SMD:C_0805_2012Metric_Pad1.18x1.45mm_HandSolder, symbol Device:C
- added C1: Cap, test_lib:C_0805_MOD, symbol test_lib:C
Connections:
- net at C2.1, C3.1, R1.1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: now also C1.1
- net at C2.2, C3.2, R1.2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: now also C1.2
Other:
- title: Test PCB - Bad PCB Lib Table -> Test PCB - Bad Lib Table
- moved on the sheet: R2
Changed lines of the file:
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@@
   (paper "USLetter")
   (title_block
-    (title "Test PCB - Bad PCB Lib Table")
-    (date "2022-04-12")
+    (title "Test PCB - Bad Lib Table")
+    (date "2022-06-04")
   )
   (junction (at 120.65 86.36) (diameter 0) (color 0 0 0 0)
@@
     (stroke (width 0) (type default) (color 0 0 0 0))
   )
-  (wire (pts (xy 127 86.36) (xy 120.65 86.36))
+  (wire (pts (xy 120.65 86.36) (xy 129.54 86.36))
     (stroke (width 0) (type default) (color 0 0 0 0))
   )
@@
     (stroke (width 0) (type default) (color 0 0 0 0))
   )
-  (wire (pts (xy 127 97.79) (xy 127 95.25))
+  (wire (pts (xy 137.16 86.36) (xy 137.16 97.79))
     (stroke (width 0) (type default) (color 0 0 0 0))
   )
-  (wire (pts (xy 120.65 97.79) (xy 127 97.79))
+  (wire (pts (xy 120.65 97.79) (xy 137.16 97.79))
     (stroke (width 0) (type default) (color 0 0 0 0))
   )
@@
     (stroke (width 0) (type default) (color 0 0 0 0))
   )
-  (wire (pts (xy 127 86.36) (xy 127 87.63))
-    (stroke (width 0) (type default) (color 0 0 0 0))
-  )
   (wire (pts (xy 92.71 95.25) (xy 92.71 97.79))
     (stroke (width 0) (type default) (color 0 0 0 0))
@@
     (stroke (width 0) (type default) (color 0 0 0 0))
   )
-  (symbol (lib_id "Device:R_US") (at 127 91.44 0) (unit 1)
+  (symbol (lib_id "Device:R_US") (at 133.35 86.36 90) (unit 1)
     (in_bom yes) (on_board yes) (fields_autoplaced)
-    (property "Reference" "R2" (id 0) (at 129.54 90.1699 0)
-      (effects (font (size 1.27 1.27)) (justify left))
-    )
-    (property "Value" "R_US" (id 1) (at 129.54 92.7099 0)
-      (effects (font (size 1.27 1.27)) (justify left))
-    )
-    (property "Footprint" "Resistor_SMD:R_4020_10251Metric_Pad1.65x5.30mm_HandSolder" (id 2) (at 128.016 91.694 90)
+    (property "Reference" "R2" (id 0) (at 133.35 80.01 90))
+    (property "Value" "R_US" (id 1) (at 133.35 82.55 90))
+    (property "Footprint" "Resistor_SMD:R_4020_10251Metric_Pad1.65x5.30mm_HandSolder" (id 2) (at 133.604 85.344 90)
       (effects (font (size 1.27 1.27)) hide)
     )
-    (property "Datasheet" "~" (id 3) (at 127 91.44 0)
+    (property "Datasheet" "~" (id 3) (at 133.35 86.36 0)
       (effects (font (size 1.27 1.27)) hide)
     )
@@
     (pin "2")
   )
-  (symbol (lib_id "Device:C") (at 82.55 91.44 0) (unit 1)
-    (in_bom yes) (on_board yes) (fields_autoplaced)
-    (property "Reference" "C1" (id 0) (at 86.36 90.1699 0)
-      (effects (font (size 1.27 1.27)) (justify left))
+  (symbol (lib_id "test_lib:C") (at 82.55 91.44 0) (mirror y) (unit 1)
+    (in_bom yes) (on_board yes)
+    (property "Reference" "C1" (id 0) (at 78.74 88.9 0)
+      (effects (font (size 1.25 1.25)) (justify right))
     )
-    (property "Value" "C" (id 1) (at 86.36 92.7099 0)
-      (effects (font (size 1.27 1.27)) (justify left))
+    (property "Value" "Cap" (id 1) (at 78.74 93.98 0)
+      (effects (font (size 1.27 1.27)) (justify right))
     )
-    (property "Footprint" "Capacitor_SMD:C_0805_2012Metric_Pad1.18x1.45mm_HandSolder" (id 2) (at 83.5152 95.25 0)
+    (property "Footprint" "test_lib:C_0805_MOD" (id 2) (at 81.5848 95.25 0)
       (effects (font (size 1.27 1.27)) hide)
     )
-    (property "Datasheet" "~" (id 3) (at 82.55 91.44 0)
+    (property "Datasheet" "www.example.com" (id 3) (at 82.55 91.44 0)
       (effects (font (size 1.27 1.27)) hide)
     )
@@
   )
   (symbol_instances
-    (path "/8247310a-de92-4616-9b08-cb00011df0ce"
-      (reference "C1") (unit 1) (value "C") (footprint "Capacitor_SMD:C_0805_2012Metric_Pad1.18x1.45mm_HandSolder")
+    (path "/7a2219c6-783a-43ff-979d-deb12dfdc6c1"
+      (reference "C1") (unit 1) (value "Cap") (footprint "test_lib:C_0805_MOD")
     )
     (path "/def4713e-f02b-49b2-8808-5569536f4eb6"
