File: test/test_project_good/test_project_good.kicad_pcb (KiCad board)
At the start: 2 copper layers, 33 x 25.4 mm, 5 parts

Commit message: Github Actions testing
Parts:
- added C4: C, Capacitor_SMD:C_0603_1608Metric, F.Cu at (147.3, 91.5)
- added C5: C, Capacitor_SMD:C_0603_1608Metric, F.Cu at (147.3, 94.0)
- C1: footprint Capacitor_SMD:C_0805_2012Metric_Pad1.18x1.45mm_HandSolder -> test_lib:C_0805_MOD
- moved C1 0.25 mm to (134.9, 88.9)
Routing:
- net Net-(C4-Pad2): track 0.00 -> 2.51 mm
- net Net-(C4-Pad1): track 0.00 -> 2.51 mm
