File: test/test_project_good/test_project_good.kicad_sch (KiCad schematic)
At the start: 5 parts

Commit message: Github Actions testing
Parts:
- removed C1: (no value), symbol Device:C
- added C1: Cap, test_lib:C_0805_MOD, symbol test_lib:C
- C2: value (none) -> C; footprint (none) -> Capacitor_SMD:C_2220_5650Metric_Pad1.97x5.40mm_HandSolder
- C3: value (none) -> C_Polarized; footprint (none) -> Capacitor_SMD:CP_Elec_6.3x5.3
- R1: value (none) -> R; footprint (none) -> Resistor_SMD:R_0612_1632Metric_Pad1.18x3.40mm_HandSolder
- R2: value (none) -> R_US; footprint (none) -> Resistor_SMD:R_4020_10251Metric_Pad1.65x5.30mm_HandSolder
Connections:
- net at C2.1, C3.1, R1.1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: now also C1.1
- net at C2.2, C3.2, R1.2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: now also C1.2
Other:
- added sheet testSheet (test.kicad_sch)
- moved on the sheet: R2
Changed lines of the file:
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@@
     (stroke (width 0) (type default) (color 0 0 0 0))
   )
-  (wire (pts (xy 127 86.36) (xy 120.65 86.36))
+  (wire (pts (xy 120.65 86.36) (xy 129.54 86.36))
     (stroke (width 0) (type default) (color 0 0 0 0))
   )
@@
     (stroke (width 0) (type default) (color 0 0 0 0))
   )
-  (wire (pts (xy 127 97.79) (xy 127 95.25))
+  (wire (pts (xy 137.16 86.36) (xy 137.16 97.79))
     (stroke (width 0) (type default) (color 0 0 0 0))
   )
-  (wire (pts (xy 120.65 97.79) (xy 127 97.79))
+  (wire (pts (xy 120.65 97.79) (xy 137.16 97.79))
     (stroke (width 0) (type default) (color 0 0 0 0))
   )
@@
     (stroke (width 0) (type default) (color 0 0 0 0))
   )
-  (wire (pts (xy 127 86.36) (xy 127 87.63))
-    (stroke (width 0) (type default) (color 0 0 0 0))
-  )
   (wire (pts (xy 92.71 95.25) (xy 92.71 97.79))
     (stroke (width 0) (type default) (color 0 0 0 0))
@@
     (stroke (width 0) (type default) (color 0 0 0 0))
   )
-  (symbol (lib_id "Device:R_US") (at 127 91.44 0) (unit 1)
+  (symbol (lib_id "Device:R_US") (at 133.35 86.36 90) (unit 1)
     (in_bom yes) (on_board yes) (fields_autoplaced)
-    (property "Reference" "R2" (id 0) (at 129.54 90.1699 0)
-      (effects (font (size 1.27 1.27)) (justify left))
-    )
-    (property "Value" "" (id 1) (at 129.54 92.7099 0)
-      (effects (font (size 1.27 1.27)) (justify left))
-    )
-    (property "Footprint" "" (id 2) (at 128.016 91.694 90)
+    (property "Reference" "R2" (id 0) (at 133.35 80.01 90))
+    (property "Value" "R_US" (id 1) (at 133.35 82.55 90))
+    (property "Footprint" "Resistor_SMD:R_4020_10251Metric_Pad1.65x5.30mm_HandSolder" (id 2) (at 133.604 85.344 90)
       (effects (font (size 1.27 1.27)) hide)
     )
-    (property "Datasheet" "~" (id 3) (at 127 91.44 0)
+    (property "Datasheet" "~" (id 3) (at 133.35 86.36 0)
       (effects (font (size 1.27 1.27)) hide)
     )
@@
     (pin "2")
   )
-  (symbol (lib_id "Device:C") (at 82.55 91.44 0) (unit 1)
-    (in_bom yes) (on_board yes) (fields_autoplaced)
-    (property "Reference" "C1" (id 0) (at 86.36 90.1699 0)
-      (effects (font (size 1.27 1.27)) (justify left))
+  (symbol (lib_id "test_lib:C") (at 82.55 91.44 0) (mirror y) (unit 1)
+    (in_bom yes) (on_board yes)
+    (property "Reference" "C1" (id 0) (at 78.74 88.9 0)
+      (effects (font (size 1.25 1.25)) (justify right))
     )
-    (property "Value" "" (id 1) (at 86.36 92.7099 0)
-      (effects (font (size 1.27 1.27)) (justify left))
+    (property "Value" "Cap" (id 1) (at 78.74 93.98 0)
+      (effects (font (size 1.27 1.27)) (justify right))
     )
-    (property "Footprint" "" (id 2) (at 83.5152 95.25 0)
+    (property "Footprint" "test_lib:C_0805_MOD" (id 2) (at 81.5848 95.25 0)
       (effects (font (size 1.27 1.27)) hide)
     )
-    (property "Datasheet" "~" (id 3) (at 82.55 91.44 0)
+    (property "Datasheet" "www.example.com" (id 3) (at 82.55 91.44 0)
       (effects (font (size 1.27 1.27)) hide)
     )
@@
       (effects (font (size 1.27 1.27)) (justify left))
     )
-    (property "Value" "" (id 1) (at 123.19 92.7099 0)
+    (property "Value" "R" (id 1) (at 123.19 92.7099 0)
       (effects (font (size 1.27 1.27)) (justify left))
     )
-    (property "Footprint" "" (id 2) (at 118.872 91.44 90)
+    (property "Footprint" "Resistor_SMD:R_0612_1632Metric_Pad1.18x3.40mm_HandSolder" (id 2) (at 118.872 91.44 90)
       (effects (font (size 1.27 1.27)) hide)
     )
@@
       (effects (font (size 1.27 1.27)) (justify left))
     )
-    (property "Value" "" (id 1) (at 96.52 92.7099 0)
+    (property "Value" "C" (id 1) (at 96.52 92.7099 0)
       (effects (font (size 1.27 1.27)) (justify left))
     )
-    (property "Footprint" "" (id 2) (at 93.6752 95.25 0)
+    (property "Footprint" "Capacitor_SMD:C_2220_5650Metric_Pad1.97x5.40mm_HandSolder" (id 2) (at 93.6752 95.25 0)
       (effects (font (size 1.27 1.27)) hide)
     )
@@
       (effects (font (size 1.27 1.27)) (justify left))
     )
-    (property "Value" "" (id 1) (at 106.68 91.8209 0)
+    (property "Value" "C_Polarized" (id 1) (at 106.68 91.8209 0)
       (effects (font (size 1.27 1.27)) (justify left))
     )
-    (property "Footprint" "" (id 2) (at 103.8352 95.25 0)
+    (property "Footprint" "Capacitor_SMD:CP_Elec_6.3x5.3" (id 2) (at 103.8352 95.25 0)
       (effects (font (size 1.27 1.27)) hide)
     )
@@
     (pin "2")
   )
+  (sheet (at 144.78 110.49) (size 17.78 11.43) (fields_autoplaced)
+    (stroke (width 0.1524) (type solid) (color 0 0 0 0))
+    (fill (color 0 0 0 0.0000))
+    (property "Sheet name" "testSheet" (id 0) (at 144.78 109.7784 0)
+      (effects (font (size 1.27 1.27)) (justify left bottom))
+    )
+    (property "Sheet file" "test.kicad_sch" (id 1) (at 144.78 122.5046 0)
+      (effects (font (size 1.27 1.27)) (justify left top))
+    )
+  )
   (sheet_instances
     (path "/" (page "1"))
+    (path "/1f72982d-1aa7-468c-a035-7868113dba21" (page "2"))
   )
   (symbol_instances
-    (path "/8247310a-de92-4616-9b08-cb00011df0ce"
-      (reference "C1") (unit 1) (value "C") (footprint "Capacitor_SMD:C_0805_2012Metric_Pad1.18x1.45mm_HandSolder")
+    (path "/7a2219c6-783a-43ff-979d-deb12dfdc6c1"
+      (reference "C1") (unit 1) (value "Cap") (footprint "test_lib:C_0805_MOD")
     )
     (path "/def4713e-f02b-49b2-8808-5569536f4eb6"
@@
       (reference "C3") (unit 1) (value "C_Polarized") (footprint "Capacitor_SMD:CP_Elec_6.3x5.3")
     )
+    (path "/1f72982d-1aa7-468c-a035-7868113dba21/a8d1da33-baba-42c6-96ac-43a85fe052af"
+      (reference "C4") (unit 1) (value "C") (footprint "Capacitor_SMD:C_0603_1608Metric")
+    )
+    (path "/1f72982d-1aa7-468c-a035-7868113dba21/cd3f1074-8efd-47e1-8c21-cab1b92a88c7"
+      (reference "C5") (unit 1) (value "C") (footprint "Capacitor_SMD:C_0603_1608Metric")
+    )
     (path "/dc90b7de-7781-4831-a51f-244db8f3a1aa"
