File: test/test_project_missing_symbol/test_project_missing_symbol.kicad_sch (KiCad schematic)
At the start: 5 parts

Commit message: Github Actions testing
Other:
- title: Test PCB - Modified Symbol -> Test PCB - All Good Libraries
Changed lines of the file:
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@@
   (paper "USLetter")
   (title_block
-    (title "Test PCB - Modified Symbol")
+    (title "Test PCB - All Good Libraries")
     (date "2022-04-12")
   )
