File: test/test_project_modified_footprint/test_project_modified_footprint.kicad_pcb (KiCad board)
At the start: 2 copper layers, 33 x 25.4 mm, 5 parts

Commit message: Github Actions testing
Parts:
- C1: footprint Capacitor_SMD:C_0805_2012Metric_Pad1.18x1.45mm_HandSolder -> test_lib:C_0805_MOD; moved to B.Cu
- moved C1 0.25 mm to (134.9, 88.9)
Routing:
- net Net-(C1-Pad2): vias 0 -> 1
- net Net-(C1-Pad1): vias 0 -> 1
